File: BalancedAudio2UnbalancedConverter.kicad_sch (KiCad schematic)
At the start: 46 parts, among them CN1 Power, CN2 XLR3, CN3 RCA, CN4 RCA, CN4 XLR3, U1 INA1650

Commit message: Board Basically done.  Just need to tweak the silkscreen.
Parts:
- added H101, H102, H103, H104: MountingHole, MountingHole:MountingHole_3.2mm_M3, symbol Mechanical:MountingHole
- CN2, CN4: Manufacturer Part Number NC3FAAH -> NC3FAAH-0; Mouser Part Number 568-NC3FAAH -> 568-NC3FAAH-O
- renumbered CN4 to CN5
Connections:
- net GND: now also U1.12 (REFA), U1.9 (REFB)
- net -VEE: now reaches L2.2
- net -VEE: now also CN1.1 (Pin_1); no longer CN1.3 (Pin_3)
- net at CN2.2: now also R14.1; no longer R15.1
- net at CN2.3: now also R15.1; no longer R14.1
- net VCC: now reaches L1.2
- net VCC: now also CN1.3 (Pin_3); no longer CN1.1 (Pin_1)
- net at CN4.2: now also R16.1; no longer R17.1
- net at CN4.3: now also R17.1; no longer R16.1
- no-connect marks 4 -> 2
Other:
- moved on the sheet: CN2, CN4

Commit message: Footprint and 3D model updates.
Parts:
- CN3, CN5: footprint ExtraFootprints:RCJ-01X-SMT -> ExtraFootprints:RCJ011SMTTR
Changed lines of the file:
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@@
       (effects (font (size 1.27 1.27)) (justify left))
     )
-    (property "Footprint" "ExtraFootprints:RCJ-01X-SMT" (id 2) (at 187.96 80.01 0)
+    (property "Footprint" "ExtraFootprints:RCJ011SMTTR" (id 2) (at 187.96 80.01 0)
       (effects (font (size 1.27 1.27)) hide)
     )
@@
       (effects (font (size 1.27 1.27)) (justify left))
     )
-    (property "Footprint" "ExtraFootprints:RCJ-01X-SMT" (id 2) (at 187.96 101.6 0)
+    (property "Footprint" "ExtraFootprints:RCJ011SMTTR" (id 2) (at 187.96 101.6 0)
       (effects (font (size 1.27 1.27)) hide)
     )
@@
     )
     (path "/4c3d3666-bc3e-4987-90c4-3ebbfcf544f3"
-      (reference "CN3") (unit 1) (value "RCA") (footprint "ExtraFootprints:RCJ-01X-SMT")
+      (reference "CN3") (unit 1) (value "RCA") (footprint "ExtraFootprints:RCJ011SMTTR")
     )
     (path "/3fd48c97-6861-4588-baab-98ec7532f17c"
@@
     )
     (path "/7325c380-b550-41b9-8e02-9dea196ee4ca"
-      (reference "CN5") (unit 1) (value "RCA") (footprint "ExtraFootprints:RCJ-01X-SMT")
+      (reference "CN5") (unit 1) (value "RCA") (footprint "ExtraFootprints:RCJ011SMTTR")
     )
     (path "/a2b98f00-1643-448a-8782-28a59494867a"
@@
     )
     (path "/4a33f9d6-fa15-4f3b-b76e-6954981c4d39/ac097fe2-7127-4be0-b57d-aabba16451ec"
-      (reference "J201") (unit 1) (value "5V In") (footprint "Connector_BarrelJack:BarrelJack_Kycon_KLDX-0202-xC_Horizontal")
+      (reference "J201") (unit 1) (value "5V In") (footprint "ExtraFootprints:KLDX0202AC")
     )
     (path "/4a33f9d6-fa15-4f3b-b76e-6954981c4d39/91b33090-e8d0-4418-9a22-5a51bf2330fb"

Commit message: Complete 3D shapes.
Parts:
- CN2: value XLR3 -> Right
- CN3: value RCA -> Right; Manufacturer Part Number RCJ-011-SMT-TR -> RCJ-012-SMT-TR; Mouser Part Number 490-RCJ-011-SMT-TR -> 490-RCJ-012-SMT-TR
- CN4: value XLR3 -> Left
- CN5: value RCA -> Left; Manufacturer Part Number RCJ-011-SMT-TR -> RCJ-013-SMT-TR; Mouser Part Number 490-RCJ-011-SMT-TR -> 490-RCJ-013-SMT-TR
Changed lines of the file:
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@@
     (in_bom yes) (on_board yes) (fields_autoplaced)
     (property "Reference" "CN2" (id 0) (at 24.13 78.74 0))
-    (property "Value" "XLR3" (id 1) (at 24.13 81.28 0))
+    (property "Value" "Right" (id 1) (at 24.13 81.28 0))
     (property "Footprint" "Connector_Audio:Jack_XLR_Neutrik_NC3FAAH_Horizontal" (id 2) (at 24.13 88.9 0)
       (effects (font (size 1.27 1.27)) hide)
@@
     (in_bom yes) (on_board yes) (fields_autoplaced)
     (property "Reference" "CN4" (id 0) (at 24.765 119.38 0))
-    (property "Value" "XLR3" (id 1) (at 24.765 121.92 0))
+    (property "Value" "Left" (id 1) (at 24.765 121.92 0))
     (property "Footprint" "Connector_Audio:Jack_XLR_Neutrik_NC3FAAH_Horizontal" (id 2) (at 24.765 129.54 0)
       (effects (font (size 1.27 1.27)) hide)
@@
       (effects (font (size 1.27 1.27)) (justify left))
     )
-    (property "Value" "RCA" (id 1) (at 190.5 81.5731 0)
+    (property "Value" "Right" (id 1) (at 190.5 81.5731 0)
       (effects (font (size 1.27 1.27)) (justify left))
     )
@@
       (effects (font (size 1.27 1.27)) hide)
     )
-    (property "Mouser Part Number" "490-RCJ-011-SMT-TR" (id 4) (at 187.96 80.01 0)
+    (property "Mouser Part Number" "490-RCJ-012-SMT-TR" (id 4) (at 187.96 80.01 0)
       (effects (font (size 1.27 1.27)) hide)
     )
@@
       (effects (font (size 1.27 1.27)) hide)
     )
-    (property "Manufacturer Part Number" "RCJ-011-SMT-TR" (id 6) (at 187.96 80.01 0)
+    (property "Manufacturer Part Number" "RCJ-012-SMT-TR" (id 6) (at 187.96 80.01 0)
       (effects (font (size 1.27 1.27)) hide)
     )
@@
       (effects (font (size 1.27 1.27)) (justify left))
     )
-    (property "Value" "RCA" (id 1) (at 190.5 102.5767 0)
+    (property "Value" "Left" (id 1) (at 190.5 102.5767 0)
       (effects (font (size 1.27 1.27)) (justify left))
     )
@@
       (effects (font (size 1.27 1.27)) hide)
     )
-    (property "Mouser Part Number" "490-RCJ-011-SMT-TR" (id 4) (at 187.96 101.6 0)
+    (property "Mouser Part Number" "490-RCJ-013-SMT-TR" (id 4) (at 187.96 101.6 0)
       (effects (font (size 1.27 1.27)) hide)
     )
@@
       (effects (font (size 1.27 1.27)) hide)
     )
-    (property "Manufacturer Part Number" "RCJ-011-SMT-TR" (id 6) (at 187.96 101.6 0)
+    (property "Manufacturer Part Number" "RCJ-013-SMT-TR" (id 6) (at 187.96 101.6 0)
       (effects (font (size 1.27 1.27)) hide)
     )
@@
     )
     (path "/15e64375-6543-4ab9-9f65-e185236d4f14"
-      (reference "CN2") (unit 1) (value "XLR3") (footprint "Connector_Audio:Jack_XLR_Neutrik_NC3FAAH_Horizontal")
+      (reference "CN2") (unit 1) (value "Right") (footprint "Connector_Audio:Jack_XLR_Neutrik_NC3FAAH_Horizontal")
     )
     (path "/4c3d3666-bc3e-4987-90c4-3ebbfcf544f3"
-      (reference "CN3") (unit 1) (value "RCA") (footprint "ExtraFootprints:RCJ011SMTTR")
+      (reference "CN3") (unit 1) (value "Right") (footprint "ExtraFootprints:RCJ011SMTTR")
     )
     (path "/3fd48c97-6861-4588-baab-98ec7532f17c"
-      (reference "CN4") (unit 1) (value "XLR3") (footprint "Connector_Audio:Jack_XLR_Neutrik_NC3FAAH_Horizontal")
+      (reference "CN4") (unit 1) (value "Left") (footprint "Connector_Audio:Jack_XLR_Neutrik_NC3FAAH_Horizontal")
     )
     (path "/7325c380-b550-41b9-8e02-9dea196ee4ca"
-      (reference "CN5") (unit 1) (value "RCA") (footprint "ExtraFootprints:RCJ011SMTTR")
+      (reference "CN5") (unit 1) (value "Left") (footprint "ExtraFootprints:RCJ011SMTTR")
     )
     (path "/a2b98f00-1643-448a-8782-28a59494867a"
