File: BalancedAudio2UnbalancedConverter.kicad_pcb (KiCad board)
At the start: 2 copper layers, 185.4 x 61 mm, 67 parts, among them CN1 Power, CN2 XLR3, CN3 RCA, CN4 XLR3, CN5 RCA, J201 5V In, J202 Power, U1 INA1650, U201 LT3582EUD-12#PBF

Commit message: Footprint and 3D model updates.
Parts:
- CN3, CN5: footprint ExtraFootprints:RCJ-01X-SMT -> ExtraFootprints:RCJ011SMTTR
- J201: footprint Connector_BarrelJack:BarrelJack_Kycon_KLDX-0202-xC_Horizontal -> ExtraFootprints:KLDX0202AC
- turned CN3 to -90 degrees
- turned CN5 to -90 degrees
Connections:
- CN3 pad 1: Net-(C6-Pad2) -> (no net)
- CN5 pad 1: Net-(C11-Pad2) -> (no net)

Commit message: Complete 3D shapes.
Parts:
- CN2: value XLR3 -> Right
- CN3: value RCA -> Right
- CN4: value XLR3 -> Left
- CN5: value RCA -> Left
Connections:
- CN3 pad 1: (no net) -> Net-(C6-Pad2)
- CN5 pad 1: (no net) -> Net-(C11-Pad2)
Changed lines of the file:
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@@
     (tags "Connector")
     (property "Manufacturer" "Same Sky")
-    (property "Manufacturer Part Number" "RCJ-011-SMT-TR")
-    (property "Mouser Part Number" "490-RCJ-011-SMT-TR")
+    (property "Manufacturer Part Number" "RCJ-012-SMT-TR")
+    (property "Mouser Part Number" "490-RCJ-012-SMT-TR")
     (property "Sheetfile" "BalancedAudio2UnbalancedConverter.kicad_sch")
     (property "Sheetname" "")
     (attr through_hole)
-    (fp_text reference "CN3" (at -0.6 0 90) (layer "F.SilkS")
+    (fp_text reference "CN3" (at 4.262 0 180) (layer "F.SilkS")
       (effects (font (size 1.27 1.27) (thickness 0.254)))
     )
-    (fp_text value "RCA" (at -0.6 0 90) (layer "F.SilkS") hide
+    (fp_text value "Right" (at 9.596 5.334 180) (layer "F.SilkS")
       (effects (font (size 1.27 1.27) (thickness 0.254)))
     )
-    (fp_text user "${REFERENCE}" (at -0.6 0 90) (layer "F.Fab")
+    (fp_text user "${REFERENCE}" (at 4.262 0 180) (layer "F.Fab")
       (effects (font (size 1.27 1.27) (thickness 0.254)))
     )
@@
     (fp_line (start -0.2 -4.15) (end -8.5 -4.15) (layer "F.Fab") (width 0.2))
     (fp_line (start 6.5 -5.5) (end 6.5 5.5) (layer "F.Fab") (width 0.2))
-    (pad "1" smd rect (at 6.2 0 270) (size 2.2 2.6) (layers "F.Cu" "F.Paste" "F.Mask"))
+    (pad "1" smd rect (at 6.2 0 270) (size 2.2 2.6) (layers "F.Cu" "F.Paste" "F.Mask")
+      (net 7 "Net-(C6-Pad2)") (pinfunction "In") (pintype "passive"))
     (pad "2" thru_hole circle (at 0 0 270) (size 2.835 2.835) (drill 1.6) (layers *.Cu *.Mask)
       (net 2 "GND") (pinfunction "Ext") (pintype "passive"))
@@
     (pad "2" smd rect (at 6 6.35 270) (size 2.2 2.5) (layers "F.Cu" "F.Paste" "F.Mask")
       (net 2 "GND") (pinfunction "Ext") (pintype "passive"))
+    (model "${KIPRJMOD}/rcj-01x-smt.step"
+      (offset (xyz 0 0 0))
+      (scale (xyz 1 1 1))
+      (rotate (xyz 0 0 90))
+    )
   )
   (footprint "MountingHole:MountingHole_3.2mm_M3" (layer "F.Cu")
@@
       (effects (font (size 1 1) (thickness 0.15)))
     )
-    (fp_text value "XLR3" (at 4.3 17.5 90) (layer "F.Fab")
+    (fp_text value "Right" (at 11.176 -11.176 180) (layer "F.SilkS")
       (effects (font (size 1 1) (thickness 0.15)))
     )
@@
     (tags "Connector")
     (property "Manufacturer" "Same Sky")
-    (property "Manufacturer Part Number" "RCJ-011-SMT-TR")
-    (property "Mouser Part Number" "490-RCJ-011-SMT-TR")
+    (property "Manufacturer Part Number" "RCJ-013-SMT-TR")
+    (property "Mouser Part Number" "490-RCJ-013-SMT-TR")
     (property "Sheetfile" "BalancedAudio2UnbalancedConverter.kicad_sch")
     (property "Sheetname" "")
     (attr through_hole)
-    (fp_text reference "CN5" (at -0.6 0 90) (layer "F.SilkS")
+    (fp_text reference "CN5" (at 3.754 -0.254 180) (layer "F.SilkS")
       (effects (font (size 1.27 1.27) (thickness 0.254)))
     )
-    (fp_text value "RCA" (at -0.6 0 90) (layer "F.SilkS") hide
+    (fp_text value "Left" (at 9.596 7.366 180) (layer "F.SilkS")
       (effects (font (size 1.27 1.27) (thickness 0.254)))
     )
-    (fp_text user "${REFERENCE}" (at -0.6 0 90) (layer "F.Fab")
+    (fp_text user "${REFERENCE}" (at 3.754 -0.254 180) (layer "F.Fab")
       (effects (font (size 1.27 1.27) (thickness 0.254)))
     )
@@
     (fp_line (start 6.5 5.5) (end -0.2 5.5) (layer "F.Fab") (width 0.2))
     (fp_line (start -0.2 -5.5) (end 6.5 -5.5) (layer "F.Fab") (width 0.2))
-    (pad "1" smd rect (at 6.2 0 270) (size 2.2 2.6) (layers "F.Cu" "F.Paste" "F.Mask"))
+    (pad "1" smd rect (at 6.2 0 270) (size 2.2 2.6) (layers "F.Cu" "F.Paste" "F.Mask")
+      (net 10 "Net-(C11-Pad2)") (pinfunction "In") (pintype "passive"))
     (pad "2" thru_hole circle (at 0 0 270) (size 2.835 2.835) (drill 1.6) (layers *.Cu *.Mask)
       (net 2 "GND") (pinfunction "Ext") (pintype "passive"))
@@
     (pad "2" smd rect (at 6 6.35 270) (size 2.2 2.5) (layers "F.Cu" "F.Paste" "F.Mask")
       (net 2 "GND") (pinfunction "Ext") (pintype "passive"))
+    (model "${KIPRJMOD}/rcj-01x-smt.step"
+      (offset (xyz 0 0 0))
+      (scale (xyz 1 1 1))
+      (rotate (xyz 0 0 90))
+    )
   )
   (footprint "Resistor_SMD:R_0805_2012Metric" (layer "F.Cu")
@@
       (effects (font (size 1 1) (thickness 0.15)))
     )
-    (fp_text value "XLR3" (at 4.3 17.5 90) (layer "F.Fab")
-      (effects (font (size 1 1) (thickness 0.15)))
-    )
+    (fp_text value "Left" (at 11.43 19.05 180) (layer "F.SilkS")
+      (effects (font (size 1 1) (thickness 0.15)))
+    )

Commit message: Minor tweaks, add 3D models of the boards.
Routing:
- net /Power Supply Board/VIN: track 1.25 -> 3.31 mm
Changed lines of the file:
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@@
   (segment (start 158.295 51.32) (end 158.485 51.32) (width 0.25) (layer "F.Cu") (net 30))
   (segment (start 162.635 49.15) (end 162.89 48.895) (width 0.25) (layer "F.Cu") (net 30))
+  (segment (start 156 53.52) (end 154.76 53.52) (width 0.5) (layer "F.Cu") (net 31))
+  (segment (start 154.76 53.52) (end 154.178 54.102) (width 0.5) (layer "F.Cu") (net 31))
   (segment (start 157.66 53.52) (end 158.496 54.356) (width 0.5) (layer "F.Cu") (net 31))
   (segment (start 157.595 53.52) (end 157.66 53.52) (width 0.25) (layer "F.Cu") (net 31))
